Commit message: Modified gitignore and URDF
Corrected a package naming error
Ignoring VIM generated files

File: packages/pepper/urdf/pepper.urdf (robot description, URDF)
Before this commit: robot pepper, 8 links, 7 joints
Links:
- link base_link: geometry visual mesh filename=package://pepper/meshes/peppercad_binary.stl scale=0.001 0.001 0.001
- link camera_link: geometry visual mesh filename=package://pepper/meshes/kinect.dae scale=0.001 0.001 0.001

Commit message: Modified URDF and Odometry

File: packages/pepper/urdf/pepper.urdf (robot description, URDF)
Before this commit: robot pepper, 8 links, 7 joints
Joints:
- joint kinect_link: origin xyz=0 0.18 0.355 rpy=0 0 1.57075 -> xyz=0.16 0 0.355 rpy=0 0 0
- joint left_motor_joint: origin xyz=-0.065 0 -0.03 rpy=0 0 0 -> xyz=0 0.065 -0.03 rpy=0 0 0
- joint left_motor_shaft_joint: origin xyz=-0.055 0 0 rpy=0 0 0 -> xyz=0 0.055 0 rpy=0 0 0
- joint right_motor_joint: origin xyz=0.065 0 -0.03 rpy=0 0 0 -> xyz=0 -0.065 -0.03 rpy=0 0 0
- joint right_motor_shaft_joint: origin xyz=0.055 0 0 rpy=0 0 0 -> xyz=0 -0.055 0 rpy=0 0 0
